File: Template Outlines/66x66/66x66.kicad_sch (KiCad schematic)
At the start: 6 parts, among them U1 RP2040, U2 MicroSense

Commit message: Updated Template, to give more of an Outline
Parts:
- removed U1: RP2040, Package_DFN_QFN:QFN-56-1EP_7x7mm_P0.4mm_EP3.2x3.2mm, symbol MCU_RaspberryPi:RP2040
- removed U2: MicroSense, Sense Board:UCA_Sense, symbol UCA Symbols:MicroSense
- added C1: 100nF, Capacitor_SMD:C_0805_2012Metric_Pad1.18x1.45mm_HandSolder, symbol Device:C
- added C2, C3: 20pF, Capacitor_SMD:C_0805_2012Metric_Pad1.18x1.45mm_HandSolder, symbol Device:C
- added J1: Conn_01x02, Connector_JST:JST_XH_B2B-XH-A_1x02_P2.50mm_Vertical, symbol Connector_Generic:Conn_01x02
- added J2: Conn_01x02, Connector_PinHeader_2.54mm:PinHeader_1x02_P2.54mm_Vertical, symbol Connector_Generic:Conn_01x02
- added J3: USB_C_Receptacle_USB2.0_14P, Connector_USB:USB_C_Receptacle_GCT_USB4105-xx-A_16P_TopMnt_Horizontal, symbol Connector:USB_C_Receptacle_USB2.0_14P
- added J4: Conn_01x03, Connector_PinSocket_2.54mm:PinSocket_1x03_P2.54mm_Vertical, symbol Connector_Generic:Conn_01x03
- added J5: Conn_01x04, Connector_PinSocket_2.54mm:PinSocket_1x04_P2.54mm_Vertical, symbol Connector_Generic:Conn_01x04
- added R1: 0R, Resistor_SMD:R_0805_2012Metric_Pad1.20x1.40mm_HandSolder, symbol Device:R
- added R10, R9: 27.4, Resistor_SMD:R_0805_2012Metric_Pad1.20x1.40mm_HandSolder, symbol Device:R
- added R2: 1k, Resistor_SMD:R_0805_2012Metric_Pad1.20x1.40mm_HandSolder, symbol Device:R
- added R3: DNP, Resistor_SMD:R_0805_2012Metric_Pad1.20x1.40mm_HandSolder, symbol Device:R
- added R4: 5.6k, Resistor_SMD:R_0805_2012Metric_Pad1.20x1.40mm_HandSolder, symbol Device:R
- added R5, R6: 5.1k, Resistor_SMD:R_0805_2012Metric_Pad1.20x1.40mm_HandSolder, symbol Device:R
- added R7, R8: 10k, Resistor_SMD:R_0805_2012Metric_Pad1.20x1.40mm_HandSolder, symbol Device:R
- added SW1: Reset, Button_Switch_SMD:SW_SPST_PTS645, symbol Switch:SW_Push
- added TP1: GND, TestPoint:TestPoint_Pad_1.0x1.0mm, symbol Connector:TestPoint
- added TP2: D-, TestPoint:TestPoint_Pad_1.0x1.0mm, symbol Connector:TestPoint
- added TP3: D+, TestPoint:TestPoint_Pad_1.0x1.0mm, symbol Connector:TestPoint
- added TP4: USB_BOOT, TestPoint:TestPoint_Pad_1.0x1.0mm, symbol Connector:TestPoint
- added TP5: USB_DET, TestPoint:TestPoint_Pad_1.0x1.0mm, symbol Connector:TestPoint
- added TP6: RST, TestPoint:TestPoint_Pad_1.0x1.0mm, symbol Connector:TestPoint
- added TP7: INT_1, TestPoint:TestPoint_Pad_1.0x1.0mm, symbol Connector:TestPoint
- added U1: W25Q128JVPIQ TR, Package_SO:SOIC-8_5.23x5.23mm_P1.27mm, symbol Memory_Flash:W25Q128JVS
- added U2: RP2040, Package_DFN_QFN:QFN-56-1EP_7x7mm_P0.4mm_EP3.2x3.2mm, symbol MCU_RaspberryPi:RP2040
- added U3: ~, Sense Board:UCA_Sense, symbol Sense:Sense_Calistated
- added Y1: 12MHz, Crystal:Crystal_SMD_3225-4Pin_3.2x2.5mm_HandSoldering, symbol Device:Crystal_GND24
- H1, H2, H3, H4: footprint MountingHole:MountingHole_3mm -> MountingHole:MountingHole_3.2mm_M3; now in the parts list
Connections:
- new net: J3.A5 (CC1), R5.1
- new net: J2.2 (Pin_2), R2.1
- new net: J3.B5 (CC2), R6.2
- new net: J3.S1 (SHIELD), R1.1
- new net +1V1: U2.23 (DVDD), U2.45 (VREG_VOUT), U2.50 (DVDD)
- new net +3V3: C1.2, J5.2 (Pin_2), R3.1, R8.2, U1.8 (VCC), U2.1 (IOVDD), U2.10 (IOVDD), U2.22 (IOVDD), U2.33 (IOVDD), U2.42 (IOVDD), U2.43 (ADC_AVDD), U2.44 (VREG_IN), U2.48 (USB_VDD), U2.49 (IOVDD), U3.6 (+3V3)
- new net ADC_0: U2.38 (GPIO26_ADC0)
- new net ADC_1: U2.39 (GPIO27_ADC1)
- new net ADC_2: U2.40 (GPIO28_ADC2)
- new net ADC_3: U2.41 (GPIO29_ADC3)
- new net Battery: J1.2 (Pin_2)
- new net CLK_GPIN0: U2.31 (GPIO20)
- new net CLK_GPOUT0: U2.32 (GPIO21)
- new net D+: J3.A6 (D+), J3.B6 (D+), R10.1, TP3.1
- new net D-: J3.A7 (D-), J3.B7 (D-), R9.1, TP2.1
- new net GND: C1.1, J1.1 (Pin_1), J2.1 (Pin_1), J3.A1 (GND), J3.A12 (GND), J3.B1 (GND), J3.B12 (GND), J4.1 (Pin_1), J5.1 (Pin_1), R1.2, R5.2, R6.1, R7.2, SW1.1, TP1.1, U1.4 (GND), U2.19 (TESTEN), U2.57 (GND), U3.4 (GND)
- new net GPIO_1: U2.3 (GPIO1)
- new net GPIO_2: U2.4 (GPIO2)
- new net GPIO_3: U2.5 (GPIO3)
- new net GPIO_4: U2.6 (GPIO4)
- new net GPIO_5: U2.7 (GPIO5)
- new net GPIO_6: U2.8 (GPIO6)
- new net GPIO_7: U2.9 (GPIO7)
- new net I2C0_SCL: J5.3 (Pin_3), U2.37 (GPIO25)
- new net I2C0_SDA: J5.4 (Pin_4), U2.36 (GPIO24)
- new net I2C1_SCL: U2.35 (GPIO23), U3.1 (SCL)
- new net I2C1_SDA: U2.34 (GPIO22), U3.3 (SDA)
- new net INT_1: TP7.1, U2.11 (GPIO8), U3.2 (INT_1)
- new net LED_GREEN: U2.14 (GPIO11)
- new net LED_RED: U2.12 (GPIO9)
- new net LED_YELLOW: U2.13 (GPIO10)
- new net QSPI_SCLK: U1.6 (CLK), U2.52 (QSPI_SCLK)
- new net QSPI_SD0: U1.5 (DI(IO0)), U2.53 (QSPI_SD0)
- new net QSPI_SD1: U1.2 (DO(IO1)), U2.55 (QSPI_SD1)
- new net QSPI_SD2: U1.3 (IO2), U2.54 (QSPI_SD2)
- new net QSPI_SD3: U1.7 (IO3), U2.51 (QSPI_SD3)
- new net QSPI_SS: R2.2, R3.2, TP4.1, U1.1 (~{CS}), U2.56 (QSPI_SS)
- new net RUN: R8.1, SW1.2, TP6.1, U2.26 (RUN)
- new net SPI0_CSn: U2.28 (GPIO17)
- new net SPI0_MISO: U2.27 (GPIO16)
- new net SPI0_MOSI: U2.30 (GPIO19)
- new net SPI0_SCK: U2.29 (GPIO18)
- new net SPI1_CSn: U2.16 (GPIO13)
- new net SPI1_MISO: U2.15 (GPIO12)
- new net SPI1_MOSI: U2.18 (GPIO15)
- new net SPI1_SCK: U2.17 (GPIO14)
- new net SWCLK: J4.3 (Pin_3), U2.24 (SWCLK)
- new net SWD: J4.2 (Pin_2), U2.25 (SWD)
- new net USB_D+: R10.2, U2.47 (USB_DP)
- new net USB_D-: R9.2, U2.46 (USB_DM)
- new net USB_DET: R4.2, R7.1, TP5.1, U2.2 (GPIO0)
- new net VBUS: J3.A4 (VBUS), J3.A9 (VBUS), J3.B4 (VBUS), J3.B9 (VBUS), R4.1
- new net XIN: U2.20 (XIN)
- new net Xout: U2.21 (XOUT)
Other:
- note added: "3V3 Regulator"
- note added: "Bypass and decoupling capacitors"
- note added: "Crystal"
- note added: "Debug Port"
- note added: "Flash"
- note added: "I2C Pullups"
- note added: "Internal 1.1v regulator bypass"
- note added: "Mounting holes"
- note added: "Power Input"
- note added: "RP2040"
- note added: "Reset Button"
- note added: "Sensors and screen"
- note added: "Status LEDs"
- note added: "USB C"
